File: MDBTMicro2840/MDBTMicro2840.kicad_sch (KiCad schematic)
At the start: 0 parts

Commit message: Update
Parts:
- added J1: Conn_01x04, Connector_PinHeader_2.54mm:PinHeader_1x04_P2.54mm_Vertical, symbol Connector_Generic:Conn_01x04
- added J2: USB_C_Receptacle_USB2.0, Connector_USB:USB_C_Receptacle_Palconn_UTC16-G, symbol Connector:USB_C_Receptacle_USB2.0
- added U1: MDBT50Q-x1MV2, MDBTMicro_library:MDBT50Q, symbol MDBTMicro_library:MDBT50Q-x1MV2
- added U2: ProMicro, MDBTMicro_library:ProMicro, symbol MDBTMicro_library:ProMicro
Connections:
- new net GND: J1.2 (Pin_2), J2.A1 (GND), J2.A12 (GND), J2.B1 (GND), J2.B12 (GND), J2.S1 (SHIELD), U1.1 (GND), U1.2 (GND), U2.3 (GND), U2.4 (GND)
- new net P0.02: U1.11 (P0.02/AIN0), U2.20 (A0)
- new net P0.03: U1.9 (P0.03/AIN1), U2.22 (14)
- new net P0.06: U1.22 (P0.06), U2.1 (TX0)
- new net P0.08: U1.24 (P0.08), U2.2 (RX1)
- new net P0.09: U1.52 (P0.09/NFC1), U2.10 (7)
- new net P0.10: U1.54 (P0.10/NFC2), U2.11 (8)
- new net P0.13: U1.37 (P0.13), U2.8 (5)
- new net P0.15: U1.39 (P0.15), U2.5 (2)
- new net P0.17: U1.41 (P0.17), U2.6 (3)
- new net P0.20: U1.44 (P0.20), U2.7 (4)
- new net P0.24: U1.48 (P0.24), U2.9 (6)
- new net P0.28: U1.13 (P0.28/AIN4), U2.23 (16)
- new net P0.29: U1.10 (P0.29/AIN5), U2.19 (A1)
- new net P0.30: U1.14 (P0.30/AIN6), U2.17 (A3)
- new net P0.31: U1.12 (P0.31/AIN7), U2.18 (A2)
- new net P1.06: U1.57 (P1.06), U2.12 (9)
- new net P1.11: U1.4 (P1.11), U2.24 (10)
- new net P1.13: U1.6 (P1.13), U2.21 (15)
- new net RESET: U1.40 (P0.18/nRESET), U2.15 (RST)
- new net SWDCLK: J1.4 (Pin_4), U1.53 (SWDCKL)
- new net SWDIO: J1.3 (Pin_3), U1.51 (SWDIO)
- new net USB_D+: J2.A6 (D+), J2.B6 (D+), U1.35 (D+)
- new net USB_D-: J2.A7 (D-), J2.B7 (D-), U1.34 (D-)
- new net VBUS: J2.A4 (VBUS), J2.A9 (VBUS), J2.B4 (VBUS), J2.B9 (VBUS), U1.32 (VBUS)
- new net VDD: J1.1 (Pin_1), U1.28 (VDD)
- no-connect marks 0 -> 2
