File: MDBTMicro2840/MDBTMicro2840.kicad_sch (KiCad schematic)
At the start: 23 parts, among them J1 USB_C_Receptacle_USB2.0, J2 SWD, U1 XC6220B331MR-G, U2 MDBT50Q-x1MV2, U3 TP4057, U4 ProMicro, X1 32.768kHz

Commit message: Update 1N5819 footprint to SOD123
Parts:
- removed C3: 10uF, Capacitor_SMD:C_0201_0603Metric, symbol Device:C_Small
- D1: footprint Diode_SMD:D_0201_0603Metric -> Diode_SMD:D_SOD-123
- renumbered C4 to C3, C5 to C4, U3 to U2, U2 to U3

Commit message: Update footprint
Parts:
- removed J2: SWD, Connector_PinHeader_1.00mm:PinHeader_1x04_P1.00mm_Vertical, symbol Connector_Generic:Conn_01x04
- removed U3: MDBT50Q-x1MV2, RF_Module:Raytac_MDBT50Q, symbol MDBTMicro_library:MDBT50Q-x1MV2
- added J2: SWD, Connector_PinHeader_1.27mm:PinHeader_1x03_P1.27mm_Vertical, symbol Connector_Generic:Conn_01x03
- added U3: MDBT50Q-1MV2, RF_Module:Raytac_MDBT50Q, symbol RF_Module:MDBT50Q-1MV2
Connections:
- net BATTERY_PIN: now also U3.20 (P0.04/AIN2)
- net GND: now also J2.1 (Pin_1), U3.1 (GND), U3.15 (GND), U3.2 (GND), U3.33 (GND), U3.55 (GND)
- net LED_PIN: now also U3.3 (P1.10)
- net P0.02: now also U3.11 (P0.02/AIN0)
- net P0.03: now also U3.9 (P0.03/AIN1)
- net P0.06: now also U3.22 (P0.06)
- net P0.08: now also U3.24 (P0.08)
- net P0.09: now also U3.52 (P0.09/NFC1)
- net P0.10: now also U3.54 (P0.10/NFC2)
- net P0.13: now also U3.37 (P0.13)
- net P0.15: now also U3.39 (P0.15)
- net P0.17: now also U3.41 (P0.17)
- net P0.20: now also U3.44 (P0.20)
- net P0.24: now also U3.48 (P0.24)
- net P0.28: now also U3.13 (P0.28/AIN4)
- net P0.29: now also U3.10 (P0.29/AIN5)
- net P0.30: now also U3.14 (P0.30/AIN6)
- net P0.31: now also U3.12 (P0.31/AIN7)
- net P1.04: now also U3.56 (P1.04)
- net P1.06: now also U3.57 (P1.06)
- net P1.11: now also U3.4 (P1.11)
- net P1.13: now also U3.6 (P1.13)
- net RESET: now also U3.40 (~{RESET}/P0.18)
- net SWCLK: now also J2.3 (Pin_3), U3.53 (SWDCLK)
- net SWDIO: now also J2.2 (Pin_2), U3.51 (SWDIO)
- net USB_D+: now also U3.35 (D+)
- net USB_D-: now also U3.34 (D-)
- net VBUS: now also U3.32 (VBUS)
- net nRF_VDD: now also U3.28 (VDD), U3.30 (VDDH)
- net at C2.2, X1.1: now also U3.17 (XL1/P0.00)
- net at C1.2, X1.2: now also U3.18 (XL2/P0.01)
Other:
- title: MDBTMicro2840 -> MDBTMicro-50Q
- moved on the sheet: C1, C2, JP1, LD2, R3, R4, R5, U4, X1

Commit message: Update sch
Parts:
- U3: value MDBT50Q-1MV2 -> MDBT50Q-x1MV2
- renumbered C2 to C1, C1 to C2
Connections:
- net at C1.2, U3.17 (XL1/P0.00): now also X1.2; no longer X1.1
- net at C2.2, U3.18 (XL2/P0.01): now also X1.1; no longer X1.2
- net P1.13 renamed P1.13/1.05
Other:
- note added: "Battery monitor"
- note added: "Compatibility Modules:"
- note added: "MDBT50Q (nRF52840/33 module)"
- note added: "P0.25"
- note added: "P1.04"
- note added: "P1.05"
- note added: "Pro Micro Board"
- note added: "SWD Interface"
- note added: "USB"
- note added: "User LED"
- note added: "for nRF52833 (MDBT50Q-x512K)"
- note added: "nRF52840 modules: (default) * MDBT50Q-1MV2 (Chip antenna) * MDBT50Q-P1MV2 (PCB antenna) * MDBT50Q-U1MV2 (External antenna) nRF52833 modules: * MDBT50Q-512K (Chip antenna) * MDBT50Q-P512K (PCB antenna) * MDBT50Q-U512K (External antenna)"
- note added: "nRF52840: JP1 Open (OFF) nRF52833: JP1 Close (ON)"
- moved on the sheet: C1, C2, J1, J2, JP1, LD2, R3, R4, R5, R6, R7, U3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
