File: MDBTMicro_50Q/MDBTMicro_50Q.kicad_sch (KiCad schematic)
At the start: 22 parts, among them J1 USB_C_Receptacle_USB2.0, J2 SWD, U1 XC6220B331MR-G, U2 TP4057, U3 MDBT50Q-x1MV2, U4 ProMicro, X1 32.768kHz

Commit message: Update footprint
Parts:
- C1, C2, C3, C4: footprint Capacitor_SMD:C_0201_0603Metric -> Capacitor_SMD:C_0603_1608Metric
- D1: footprint Diode_SMD:D_SOD-123 -> Diode_SMD:D_SOD-323F
- LD1: value RED -> Charging; footprint LED_SMD:LED_0201_0603Metric -> LED_SMD:LED_0603_1608Metric
- LD2: value BLUE -> User; footprint LED_SMD:LED_0201_0603Metric -> LED_SMD:LED_0603_1608Metric
- R1, R2, R3, R4, R5, R6, R7: footprint Resistor_SMD:R_0201_0603Metric -> Resistor_SMD:R_0603_1608Metric
- X1: footprint Crystal:Crystal_SMD_3215-2Pin_3.2x1.5mm -> Crystal:Crystal_SMD_MicroCrystal_CM9V-T1A-2Pin_1.6x1.0mm
Other:
- note added: "LiPo Charger"
- note removed: "LiPo Charging"
Changed lines of the file:
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@@
     (effects (font (size 1.27 1.27)) (justify left bottom))
   )
-  (text "LiPo Charging" (at 27.94 165.1 0)
+  (text "LiPo Charger" (at 27.94 165.1 0)
     (effects (font (size 1.27 1.27)) (justify left bottom))
   )
@@
     (property "Reference" "C1" (id 0) (at 115.57 33.02 90))
     (property "Value" "12pF" (id 1) (at 115.57 35.56 90))
-    (property "Footprint" "Capacitor_SMD:C_0201_0603Metric" (id 2) (at 115.57 38.1 0)
+    (property "Footprint" "Capacitor_SMD:C_0603_1608Metric" (id 2) (at 115.57 38.1 0)
       (effects (font (size 1.27 1.27)) hide)
     )
@@
     (property "Reference" "D1" (id 0) (at 40.9575 137.16 0))
     (property "Value" "1N5819" (id 1) (at 40.9575 139.7 0))
-    (property "Footprint" "Diode_SMD:D_SOD-123" (id 2) (at 40.64 139.065 0)
+    (property "Footprint" "Diode_SMD:D_SOD-323F" (id 2) (at 40.64 139.065 0)
       (effects (font (size 1.27 1.27)) hide)
     )
@@
       (effects (font (size 1.27 1.27)) (justify right))
     )
-    (property "Footprint" "Crystal:Crystal_SMD_3215-2Pin_3.2x1.5mm" (id 2) (at 111.76 41.91 0)
+    (property "Footprint" "Crystal:Crystal_SMD_MicroCrystal_CM9V-T1A-2Pin_1.6x1.0mm" (id 2) (at 111.76 41.91 0)
       (effects (font (size 1.27 1.27)) hide)
     )
@@
     (property "Reference" "R5" (id 0) (at 118.11 142.24 90))
     (property "Value" "1k" (id 1) (at 118.11 144.78 90))
-    (property "Footprint" "Resistor_SMD:R_0201_0603Metric" (id 2) (at 118.11 147.32 0)
+    (property "Footprint" "Resistor_SMD:R_0603_1608Metric" (id 2) (at 118.11 147.32 0)
       (effects (font (size 1.27 1.27)) hide)
     )
@@
     (property "Reference" "R7" (id 0) (at 257.81 36.83 90))
     (property "Value" "5.1k" (id 1) (at 264.16 36.83 90))
-    (property "Footprint" "Resistor_SMD:R_0201_0603Metric" (id 2) (at 260.35 38.1 0)
+    (property "Footprint" "Resistor_SMD:R_0603_1608Metric" (id 2) (at 260.35 38.1 0)
       (effects (font (size 1.27 1.27)) hide)
     )
@@
     (property "Reference" "C3" (id 0) (at 41.91 148.59 0))
     (property "Value" "10uF" (id 1) (at 40.64 151.13 0))
-    (property "Footprint" "Capacitor_SMD:C_0201_0603Metric" (id 2) (at 44.45 149.86 0)
+    (property "Footprint" "Capacitor_SMD:C_0603_1608Metric" (id 2) (at 44.45 149.86 0)
       (effects (font (size 1.27 1.27)) hide)
     )
@@
     (property "Reference" "C4" (id 0) (at 74.93 148.59 0))
     (property "Value" "10uF" (id 1) (at 76.2 151.13 0))
-    (property "Footprint" "Capacitor_SMD:C_0201_0603Metric" (id 2) (at 72.39 149.86 0)
+    (property "Footprint" "Capacitor_SMD:C_0603_1608Metric" (id 2) (at 72.39 149.86 0)
       (effects (font (size 1.27 1.27)) hide)
     )
@@
     (in_bom yes) (on_board yes)
     (property "Reference" "LD2" (id 0) (at 110.49 142.24 0))
-    (property "Value" "BLUE" (id 1) (at 110.49 144.78 0))
-    (property "Footprint" "LED_SMD:LED_0201_0603Metric" (id 2) (at 110.49 147.32 0)
+    (property "Value" "User" (id 1) (at 110.49 144.78 0))
+    (property "Footprint" "LED_SMD:LED_0603_1608Metric" (id 2) (at 110.49 147.32 0)
       (effects (font (size 1.27 1.27)) hide)
     )
@@
     (in_bom yes) (on_board yes)
     (property "Reference" "LD1" (id 0) (at 57.15 167.64 0))
-    (property "Value" "RED" (id 1) (at 57.15 170.18 0))
-    (property "Footprint" "LED_SMD:LED_0201_0603Metric" (id 2) (at 57.15 172.72 0)
+    (property "Value" "Charging" (id 1) (at 57.15 168.91 0))
+    (property "Footprint" "LED_SMD:LED_0603_1608Metric" (id 2) (at 57.15 172.72 0)
       (effects (font (size 1.27 1.27)) hide)
     )
@@
     (property "Reference" "R6" (id 0) (at 257.81 34.29 90))
     (property "Value" "5.1k" (id 1) (at 264.16 34.29 90))
-    (property "Footprint" "Resistor_SMD:R_0201_0603Metric" (id 2) (at 260.35 35.56 0)
+    (property "Footprint" "Resistor_SMD:R_0603_1608Metric" (id 2) (at 260.35 35.56 0)
       (effects (font (size 1.27 1.27)) hide)
     )
@@
     (property "Reference" "R3" (id 0) (at 116.84 175.26 0))
     (property "Value" "820k" (id 1) (at 118.11 177.8 0))
-    (property "Footprint" "Resistor_SMD:R_0201_0603Metric" (id 2) (at 114.3 176.53 0)
+    (property "Footprint" "Resistor_SMD:R_0603_1608Metric" (id 2) (at 114.3 176.53 0)
       (effects (font (size 1.27 1.27)) hide)
     )
@@
     (property "Reference" "C2" (id 0) (at 115.57 50.8 90))
     (property "Value" "12pF" (id 1) (at 115.57 48.26 90))
-    (property "Footprint" "Capacitor_SMD:C_0201_0603Metric" (id 2) (at 115.57 45.72 0)
+    (property "Footprint" "Capacitor_SMD:C_0603_1608Metric" (id 2) (at 115.57 45.72 0)
       (effects (font (size 1.27 1.27)) hide)
     )
@@
     (property "Reference" "R2" (id 0) (at 59.69 182.88 90))
     (property "Value" "Rprog" (id 1) (at 59.69 180.34 90))
-    (property "Footprint" "Resistor_SMD:R_0201_0603Metric" (id 2) (at 59.69 177.8 0)
+    (property "Footprint" "Resistor_SMD:R_0603_1608Metric" (id 2) (at 59.69 177.8 0)
       (effects (font (size 1.27 1.27)) hide)
     )
@@
     (property "Reference" "R4" (id 0) (at 116.84 182.88 0))
     (property "Value" "2M" (id 1) (at 116.84 185.42 0))
-    (property "Footprint" "Resistor_SMD:R_0201_0603Metric" (id 2) (at 114.3 184.15 0)
+    (property "Footprint" "Resistor_SMD:R_0603_1608Metric" (id 2) (at 114.3 184.15 0)
       (effects (font (size 1.27 1.27)) hide)
     )
@@
     (property "Reference" "R1" (id 0) (at 50.8 167.64 90))
     (property "Value" "1k" (id 1) (at 50.8 170.18 90))
-    (property "Footprint" "Resistor_SMD:R_0201_0603Metric" (id 2) (at 50.8 172.72 0)
+    (property "Footprint" "Resistor_SMD:R_0603_1608Metric" (id 2) (at 50.8 172.72 0)
       (effects (font (size 1.27 1.27)) hide)
     )
@@
     )
     (path "/13fd9f4e-8aad-4de4-885e-e5a7e914d2fe"
-      (reference "C1") (unit 1) (value "12pF") (footprint "Capacitor_SMD:C_0201_0603Metric")
+      (reference "C1") (unit 1) (value "12pF") (footprint "Capacitor_SMD:C_0603_1608Metric")
     )
     (path "/be5a0549-0f50-4ef7-86a4-0fafffa63054"
-      (reference "C2") (unit 1) (value "12pF") (footprint "Capacitor_SMD:C_0201_0603Metric")
+      (reference "C2") (unit 1) (value "12pF") (footprint "Capacitor_SMD:C_0603_1608Metric")
     )
     (path "/831ed25b-06ff-404b-9c1b-d891147fcc2a"
-      (reference "C3") (unit 1) (value "10uF") (footprint "Capacitor_SMD:C_0201_0603Metric")
+      (reference "C3") (unit 1) (value "10uF") (footprint "Capacitor_SMD:C_0603_1608Metric")
     )
     (path "/a7132da1-f35b-44d1-bdff-4ad86be7eba9"
-      (reference "C4") (unit 1) (value "10uF") (footprint "Capacitor_SMD:C_0201_0603Metric")
+      (reference "C4") (unit 1) (value "10uF") (footprint "Capacitor_SMD:C_0603_1608Metric")
     )
     (path "/1db18ded-c5e4-4e36-b70e-e5c719fb0604"
-      (reference "D1") (unit 1) (value "1N5819") (footprint "Diode_SMD:D_SOD-123")
+      (reference "D1") (unit 1) (value "1N5819") (footprint "Diode_SMD:D_SOD-323F")
     )
     (path "/4b8db155-c4c2-4b60-8a6b-2451525c938a"
@@
     )
     (path "/b267cf09-7445-4107-8705-5aaf40fe91db"
-      (reference "LD1") (unit 1) (value "RED") (footprint "LED_SMD:LED_0201_0603Metric")
+      (reference "LD1") (unit 1) (value "Charging") (footprint "LED_SMD:LED_0603_1608Metric")
     )
     (path "/b24ca40b-051b-4aec-90a7-31ee28fccb04"
-      (reference "LD2") (unit 1) (value "BLUE") (footprint "LED_SMD:LED_0201_0603Metric")
+      (reference "LD2") (unit 1) (value "User") (footprint "LED_SMD:LED_0603_1608Metric")
     )
     (path "/c6a618c1-d3b0-41f6-a9e3-27013f2fb0fc"
-      (reference "R1") (unit 1) (value "1k") (footprint "Resistor_SMD:R_0201_0603Metric")
+      (reference "R1") (unit 1) (value "1k") (footprint "Resistor_SMD:R_0603_1608Metric")
     )
     (path "/c1b357c5-9864-4302-86e9-0f2bce3c7921"
-      (reference "R2") (unit 1) (value "Rprog") (footprint "Resistor_SMD:R_0201_0603Metric")
+      (reference "R2") (unit 1) (value "Rprog") (footprint "Resistor_SMD:R_0603_1608Metric")
     )
     (path "/bddd06af-956e-4243-b181-c10236fb1923"
-      (reference "R3") (unit 1) (value "820k") (footprint "Resistor_SMD:R_0201_0603Metric")
+      (reference "R3") (unit 1) (value "820k") (footprint "Resistor_SMD:R_0603_1608Metric")
     )
     (path "/c63ae977-b30d-41fe-ac4e-ae8e7877b3c7"
-      (reference "R4") (unit 1) (value "2M") (footprint "Resistor_SMD:R_0201_0603Metric")
+      (reference "R4") (unit 1) (value "2M") (footprint "Resistor_SMD:R_0603_1608Metric")
     )
     (path "/52a6a806-64e4-4d76-ac2c-1ba2786d9d97"
-      (reference "R5") (unit 1) (value "1k") (footprint "Resistor_SMD:R_0201_0603Metric")
+      (reference "R5") (unit 1) (value "1k") (footprint "Resistor_SMD:R_0603_1608Metric")
     )
     (path "/b6b8c858-1736-47a7-a5a9-2161c3c217d6"
-      (reference "R6") (unit 1) (value "5.1k") (footprint "Resistor_SMD:R_0201_0603Metric")
+      (reference "R6") (unit 1) (value "5.1k") (footprint "Resistor_SMD:R_0603_1608Metric")
     )
     (path "/63f345a0-ca21-45a2-8405-fdefe13e2ca5"
-      (reference "R7") (unit 1) (value "5.1k") (footprint "Resistor_SMD:R_0201_0603Metric")
+      (reference "R7") (unit 1) (value "5.1k") (footprint "Resistor_SMD:R_0603_1608Metric")
     )
     (path "/e85cc31d-49c1-43d6-b1b8-a9b93729e243"
@@
     )
     (path "/3bb0dd81-bdfe-4040-a6e3-115f5c1fc0f7"
-      (reference "X1") (unit 1) (value "32.768kHz") (footprint "Crystal:Crystal_SMD_3215-2Pin_3.2x1.5mm")
-    )
-  )
+      (reference "X1") (unit 1) (value "32.768kHz") (footprint "Crystal:Crystal_SMD_MicroCrystal_CM9V-T1A-2Pin_1.6x1.0mm")
+    )
+  )

Commit message: Update sch and pcb
Connections:
- net VBAT: no longer U4.13 (RAW)
- net VBUS: now also U4.13 (RAW)
Changed lines of the file:
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@@
+    )
+  )
+  (global_label "VBUS" (shape input) (at 187.96 33.02 0) (fields_autoplaced)
+    (effects (font (size 1.27 1.27)) (justify left))
+    (property "Intersheet References" "${INTERSHEET_REFS}" (id 0) (at 195.2717 32.9406 0)
+      (effects (font (size 1.27 1.27)) (justify left) hide)
     )
   )
@@
       (effects (font (size 1.27 1.27)) (justify left) hide)
     )
-  )
-  (global_label "VBAT" (shape input) (at 187.96 33.02 0) (fields_autoplaced)
-    (effects (font (size 1.27 1.27)) (justify left))
-    (property "Intersheet References" "${INTERSHEET_REFS}" (id 0) (at 194.7879 32.9406 0)
-      (effects (font (size 1.27 1.27)) (justify left) hide)
-    )
