File: MDBTMicro_50Q/MDBTMicro_50Q.kicad_sch (KiCad schematic)
At the start: 22 parts, among them J1 USB_C_Receptacle_USB2.0, J2 SWD, U1 XC6220B331MR-G, U2 TP4057, U3 MDBT50Q-x1MV2, U4 ProMicro, X1 32.768kHz

Commit message: Update
Parts:
- removed C3, C4: 10uF, Capacitor_SMD:C_0603_1608Metric, symbol Device:C_Small
- removed J2: SWD, Connector_PinHeader_1.27mm:PinHeader_1x03_P1.27mm_Vertical, symbol Connector_Generic:Conn_01x03
- added C1, C2: 1uF, Capacitor_SMD:C_0402_1005Metric, symbol Device:C_Small
- added Q1, Q2: AO3407, Package_TO_SOT_SMD:SOT-23, symbol Transistor_FET:AO3401A
- added R1: 100k, Resistor_SMD:R_0402_1005Metric, symbol Device:R_Small_US
- added R7: 2M, Resistor_SMD:R_0402_1005Metric, symbol Device:R_Small_US
- added TP1, TP2, TP3, TP4, TP5, TP6, TP7: TestPoint, TestPoint:TestPoint_Pad_D1.0mm, symbol Connector:TestPoint
- added TP10: SWCLK, TestPoint:TestPoint_Pad_D1.0mm, symbol Connector:TestPoint
- added TP8: GND, TestPoint:TestPoint_Pad_D1.0mm, symbol Connector:TestPoint
- added TP9: SWDIO, TestPoint:TestPoint_Pad_D1.0mm, symbol Connector:TestPoint
- C3: renamed from C1; footprint Capacitor_SMD:C_0603_1608Metric -> Capacitor_SMD:C_0402_1005Metric
- C4: renamed from C2; footprint Capacitor_SMD:C_0603_1608Metric -> Capacitor_SMD:C_0402_1005Metric
- J1: renamed from U4; value ProMicro -> ProMicro Pinout
- LD1, LD2: footprint LED_SMD:LED_0603_1608Metric -> LED_SMD:LED_0402_1005Metric
- R2: renamed from R1; footprint Resistor_SMD:R_0603_1608Metric -> Resistor_SMD:R_0402_1005Metric
- R3: renamed from R2; footprint Resistor_SMD:R_0603_1608Metric -> Resistor_SMD:R_0402_1005Metric
- R4: renamed from R5; footprint Resistor_SMD:R_0603_1608Metric -> Resistor_SMD:R_0402_1005Metric
- R5: renamed from R3; footprint Resistor_SMD:R_0603_1608Metric -> Resistor_SMD:R_0402_1005Metric
- R6: renamed from R4; footprint Resistor_SMD:R_0603_1608Metric -> Resistor_SMD:R_0402_1005Metric
- R8: renamed from R6; footprint Resistor_SMD:R_0603_1608Metric -> Resistor_SMD:R_0402_1005Metric
- R9: renamed from R7; footprint Resistor_SMD:R_0603_1608Metric -> Resistor_SMD:R_0402_1005Metric
- U1: footprint MDBTMicro_library:SOT-25-5 -> Package_TO_SOT_SMD:SOT-23-5
- X1: footprint Crystal:Crystal_SMD_MicroCrystal_CM9V-T1A-2Pin_1.6x1.0mm -> Crystal:Crystal_SMD_MicroCrystal_CC7V-T1A-2Pin_3.2x1.5mm
- renumbered J1 to J2, U3 to U2, U2 to U3
Connections:
- net GND: now also C1.2, C2.2, R1.2, R7.2, TP8.1
- net SWCLK: now also TP10.1
- net SWDIO: now also TP9.1
- net VBAT: now also Q1.3 (D); no longer D1.2 (A)
- net VBUS: now also D1.2 (A), Q1.1 (G), R1.1; no longer D1.1 (K), U1.1 (VIN), U1.3 (CE)
- net nRF_VDD: now also C2.1, Q2.2 (S); no longer J1.16 (VCC)
- net P0.05: now reaches U2.21 (P0.05/AIN3)
- net P0.05: now also TP5.1
- net P0.07: now reaches U2.23 (TRACECLK/P0.07)
- net P0.07: now also TP4.1
- net POWER_PIN: now reaches U2.26 (TRACEDATA3/P1.09)
- net POWER_PIN: now also Q2.1 (G), R7.1
- net P0.11: now reaches U2.27 (TRACEDATA2/P0.11)
- net P0.11: now also TP7.1
- net P0.12: now reaches U2.29 (TRACEDATA1/P0.12)
- net P0.12: now also TP6.1
- net P1.12: now reaches U2.5 (P1.12)
- net P1.12: now also TP1.1
- net P1.14: now reaches U2.7 (P1.14)
- net P1.14: now also TP2.1
- net P1.15: now reaches U2.8 (P1.15)
- net P1.15: now also TP3.1
- net P1.13/1.05 renamed P1.13
- new net: C1.1, D1.1 (K), Q1.2 (S), U1.1 (VIN), U1.3 (CE)
- new net EXT_VCC: J1.16 (VCC), Q2.3 (D)
- no-connect marks 28 -> 20
Other:
- note added: "Battery Monitor"
- note added: "P0.19"
- note added: "P0.23"
- note added: "P1.03"
- note added: "Power Switch"
- note added: "Pro Micro Board Pinout"
- note removed: "Battery monitor"
- note removed: "Compatibility Modules:"
- note removed: "Pro Micro Board"
- note removed: "nRF52840 modules: (default) * MDBT50Q-1MV2 (Chip antenna) * MDBT50Q-P1MV2 (PCB antenna) * MDBT50Q-U1MV2 (External antenna) nRF52833 modules: * MDBT50Q-512K (Chip antenna) * MDBT50Q-P512K (PCB antenna) * MDBT50Q-U512K (External antenna)"
- moved on the sheet: C3, C4, D1, J1, J2, JP1, LD1, LD2, R2, R3, R4, R5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
