File: MDBTMicro_50Q/MDBTMicro_50Q.kicad_sch (KiCad schematic)
At the start: 35 parts, among them J1 ProMicro Pinout, J2 USB_C_Receptacle_USB2.0, Q1 AO3407, Q2 AO3407, U1 XC6220B331MR-G, U2 MDBT50Q-x1MV2, U3 TP4057, X1 32.768kHz

Commit message: Update 1.2
Parts:
- added LD3: Green, LED_SMD:LED_0402_1005Metric, symbol Device:LED
- added R5: 1k, Resistor_SMD:R_0402_1005Metric, symbol Device:R_Small_US
- J1: footprint MDBTMicro_library:ProMicro -> MDBTMicro_library:ProMicro board pinout
- LD1: value Charging -> Red
- LD2: value User -> Blue
- renumbered R9 to R10, R5 to R6, R6 to R7, R7 to R8, R8 to R9
Connections:
- net GND: now also R5.1
- net VBUS: now also LD3.2 (A)
- new net: LD3.1 (K), R5.2
Other:
- note added: "LED"
- note removed: "User LED"
- moved on the sheet: LD2, R4

Commit message: Update 1.3
Parts:
- C1, C2, C3, C4: footprint Capacitor_SMD:C_0402_1005Metric -> Capacitor_SMD:C_0603_1608Metric
- LD1, LD2: footprint LED_SMD:LED_0402_1005Metric -> LED_SMD:LED_0603_1608Metric
- R1, R10, R2, R3, R4, R6, R7, R8, R9: footprint Resistor_SMD:R_0402_1005Metric -> Resistor_SMD:R_0603_1608Metric
Changed lines of the file:
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@@
   (title_block
     (title "MDBTMicro-50Q")
-    (date "2022-10-16")
-    (rev "1.2")
+    (date "2022-10-18")
+    (rev "1.3")
     (comment 1 "For Raytac MDBT50Q (Nordic nRF52840/33 module)")
     (comment 2 "MIT License (OSHW)")
@@
     (property "Reference" "C3" (id 0) (at 115.57 43.18 90))
     (property "Value" "12pF" (id 1) (at 115.57 45.72 90))
-    (property "Footprint" "Capacitor_SMD:C_0402_1005Metric" (id 2) (at 115.57 48.26 0)
+    (property "Footprint" "Capacitor_SMD:C_0603_1608Metric" (id 2) (at 115.57 48.26 0)
       (effects (font (size 1.27 1.27)) hide)
     )
@@
     (property "Reference" "C1" (id 0) (at 50.8 175.26 0))
     (property "Value" "1uF" (id 1) (at 52.07 177.8 0))
-    (property "Footprint" "Capacitor_SMD:C_0402_1005Metric" (id 2) (at 54.61 175.26 0)
+    (property "Footprint" "Capacitor_SMD:C_0603_1608Metric" (id 2) (at 54.61 175.26 0)
       (effects (font (size 1.27 1.27)) hide)
     )
@@
     (property "Reference" "R1" (id 0) (at 31.75 175.26 90))
     (property "Value" "100k" (id 1) (at 34.29 175.26 90))
-    (property "Footprint" "Resistor_SMD:R_0402_1005Metric" (id 2) (at 36.83 175.26 0)
+    (property "Footprint" "Resistor_SMD:R_0603_1608Metric" (id 2) (at 36.83 175.26 0)
       (effects (font (size 1.27 1.27)) hide)
     )
@@
     (property "Reference" "R4" (id 0) (at 149.86 135.89 0))
     (property "Value" "1k" (id 1) (at 149.86 133.35 0))
-    (property "Footprint" "Resistor_SMD:R_0402_1005Metric" (id 2) (at 146.05 134.62 0)
+    (property "Footprint" "Resistor_SMD:R_0603_1608Metric" (id 2) (at 146.05 134.62 0)
       (effects (font (size 1.27 1.27)) hide)
     )
@@
     (property "Reference" "R10" (id 0) (at 257.81 41.91 90))
     (property "Value" "5.1k" (id 1) (at 264.16 41.91 90))
-    (property "Footprint" "Resistor_SMD:R_0402_1005Metric" (id 2) (at 260.35 43.18 0)
+    (property "Footprint" "Resistor_SMD:R_0603_1608Metric" (id 2) (at 260.35 43.18 0)
       (effects (font (size 1.27 1.27)) hide)
     )
@@
     (property "Reference" "R8" (id 0) (at 243.84 133.35 90))
     (property "Value" "2M" (id 1) (at 246.38 133.35 90))
-    (property "Footprint" "Resistor_SMD:R_0402_1005Metric" (id 2) (at 248.92 133.35 0)
+    (property "Footprint" "Resistor_SMD:R_0603_1608Metric" (id 2) (at 248.92 133.35 0)
       (effects (font (size 1.27 1.27)) hide)
     )
@@
     (property "Reference" "C2" (id 0) (at 80.01 175.26 0))
     (property "Value" "1uF" (id 1) (at 81.28 177.8 0))
-    (property "Footprint" "Capacitor_SMD:C_0402_1005Metric" (id 2) (at 83.82 175.26 0)
+    (property "Footprint" "Capacitor_SMD:C_0603_1608Metric" (id 2) (at 83.82 175.26 0)
       (effects (font (size 1.27 1.27)) hide)
     )
@@
     (property "Reference" "LD2" (id 0) (at 149.86 127 90))
     (property "Value" "Blue" (id 1) (at 149.86 124.46 90))
-    (property "Footprint" "LED_SMD:LED_0402_1005Metric" (id 2) (at 146.05 127 0)
+    (property "Footprint" "LED_SMD:LED_0603_1608Metric" (id 2) (at 146.05 127 0)
       (effects (font (size 1.27 1.27)) hide)
     )
@@
     (property "Reference" "LD1" (id 0) (at 133.35 158.75 0))
     (property "Value" "Red" (id 1) (at 133.35 161.29 0))
-    (property "Footprint" "LED_SMD:LED_0402_1005Metric" (id 2) (at 133.35 163.83 0)
+    (property "Footprint" "LED_SMD:LED_0603_1608Metric" (id 2) (at 133.35 163.83 0)
       (effects (font (size 1.27 1.27)) hide)
     )
@@
     (property "Reference" "R9" (id 0) (at 257.81 39.37 90))
     (property "Value" "5.1k" (id 1) (at 264.16 39.37 90))
-    (property "Footprint" "Resistor_SMD:R_0402_1005Metric" (id 2) (at 260.35 40.64 0)
+    (property "Footprint" "Resistor_SMD:R_0603_1608Metric" (id 2) (at 260.35 40.64 0)
       (effects (font (size 1.27 1.27)) hide)
     )
@@
     (property "Reference" "R6" (id 0) (at 200.66 124.46 0))
     (property "Value" "820k" (id 1) (at 201.93 127 0))
-    (property "Footprint" "Resistor_SMD:R_0402_1005Metric" (id 2) (at 198.12 125.73 0)
+    (property "Footprint" "Resistor_SMD:R_0603_1608Metric" (id 2) (at 198.12 125.73 0)
       (effects (font (size 1.27 1.27)) hide)
     )
@@
     (property "Reference" "C4" (id 0) (at 115.57 60.96 90))
     (property "Value" "12pF" (id 1) (at 115.57 58.42 90))
-    (property "Footprint" "Capacitor_SMD:C_0402_1005Metric" (id 2) (at 115.57 55.88 0)
+    (property "Footprint" "Capacitor_SMD:C_0603_1608Metric" (id 2) (at 115.57 55.88 0)
       (effects (font (size 1.27 1.27)) hide)
     )
@@
     (property "Reference" "R3" (id 0) (at 135.89 173.99 90))
     (property "Value" "Rprog" (id 1) (at 135.89 171.45 90))
-    (property "Footprint" "Resistor_SMD:R_0402_1005Metric" (id 2) (at 135.89 168.91 0)
+    (property "Footprint" "Resistor_SMD:R_0603_1608Metric" (id 2) (at 135.89 168.91 0)
       (effects (font (size 1.27 1.27)) hide)
     )
@@
     (property "Reference" "R7" (id 0) (at 200.66 132.08 0))
     (property "Value" "2M" (id 1) (at 200.66 134.62 0))
-    (property "Footprint" "Resistor_SMD:R_0402_1005Metric" (id 2) (at 198.12 133.35 0)
+    (property "Footprint" "Resistor_SMD:R_0603_1608Metric" (id 2) (at 198.12 133.35 0)
       (effects (font (size 1.27 1.27)) hide)
     )
@@
     (property "Reference" "R2" (id 0) (at 127 158.75 90))
     (property "Value" "1k" (id 1) (at 127 161.29 90))
-    (property "Footprint" "Resistor_SMD:R_0402_1005Metric" (id 2) (at 127 163.83 0)
+    (property "Footprint" "Resistor_SMD:R_0603_1608Metric" (id 2) (at 127 163.83 0)
       (effects (font (size 1.27 1.27)) hide)
     )
@@
     )
     (path "/33f8d1c9-98b7-46f4-b122-b574190e8956"
-      (reference "C1") (unit 1) (value "1uF") (footprint "Capacitor_SMD:C_0402_1005Metric")
+      (reference "C1") (unit 1) (value "1uF") (footprint "Capacitor_SMD:C_0603_1608Metric")
     )
     (path "/b065d225-1553-41e6-93c1-047b538bd71f"
-      (reference "C2") (unit 1) (value "1uF") (footprint "Capacitor_SMD:C_0402_1005Metric")
+      (reference "C2") (unit 1) (value "1uF") (footprint "Capacitor_SMD:C_0603_1608Metric")
     )
     (path "/13fd9f4e-8aad-4de4-885e-e5a7e914d2fe"
-      (reference "C3") (unit 1) (value "12pF") (footprint "Capacitor_SMD:C_0402_1005Metric")
+      (reference "C3") (unit 1) (value "12pF") (footprint "Capacitor_SMD:C_0603_1608Metric")
     )
     (path "/be5a0549-0f50-4ef7-86a4-0fafffa63054"
-      (reference "C4") (unit 1) (value "12pF") (footprint "Capacitor_SMD:C_0402_1005Metric")
+      (reference "C4") (unit 1) (value "12pF") (footprint "Capacitor_SMD:C_0603_1608Metric")
     )
     (path "/1db18ded-c5e4-4e36-b70e-e5c719fb0604"
@@
     )
     (path "/b267cf09-7445-4107-8705-5aaf40fe91db"
-      (reference "LD1") (unit 1) (value "Red") (footprint "LED_SMD:LED_0402_1005Metric")
+      (reference "LD1") (unit 1) (value "Red") (footprint "LED_SMD:LED_0603_1608Metric")
     )
     (path "/b24ca40b-051b-4aec-90a7-31ee28fccb04"
-      (reference "LD2") (unit 1) (value "Blue") (footprint "LED_SMD:LED_0402_1005Metric")
+      (reference "LD2") (unit 1) (value "Blue") (footprint "LED_SMD:LED_0603_1608Metric")
     )
     (path "/c60794a5-e0bc-4a2f-9e0d-4114d23ce17e"
@@
     )
     (path "/42e64acb-2ae0-46da-b1ed-906168be6011"
-      (reference "R1") (unit 1) (value "100k") (footprint "Resistor_SMD:R_0402_1005Metric")
+      (reference "R1") (unit 1) (value "100k") (footprint "Resistor_SMD:R_0603_1608Metric")
     )
     (path "/c6a618c1-d3b0-41f6-a9e3-27013f2fb0fc"
-      (reference "R2") (unit 1) (value "1k") (footprint "Resistor_SMD:R_0402_1005Metric")
+      (reference "R2") (unit 1) (value "1k") (footprint "Resistor_SMD:R_0603_1608Metric")
     )
     (path "/c1b357c5-9864-4302-86e9-0f2bce3c7921"
-      (reference "R3") (unit 1) (value "Rprog") (footprint "Resistor_SMD:R_0402_1005Metric")
+      (reference "R3") (unit 1) (value "Rprog") (footprint "Resistor_SMD:R_0603_1608Metric")
     )
     (path "/52a6a806-64e4-4d76-ac2c-1ba2786d9d97"
-      (reference "R4") (unit 1) (value "1k") (footprint "Resistor_SMD:R_0402_1005Metric")
+      (reference "R4") (unit 1) (value "1k") (footprint "Resistor_SMD:R_0603_1608Metric")
     )
     (path "/b3fce5d5-8864-47ee-abb8-af5752aa6870"
@@
     )
     (path "/bddd06af-956e-4243-b181-c10236fb1923"
-      (reference "R6") (unit 1) (value "820k") (footprint "Resistor_SMD:R_0402_1005Metric")
+      (reference "R6") (unit 1) (value "820k") (footprint "Resistor_SMD:R_0603_1608Metric")
     )
     (path "/c63ae977-b30d-41fe-ac4e-ae8e7877b3c7"
-      (reference "R7") (unit 1) (value "2M") (footprint "Resistor_SMD:R_0402_1005Metric")
+      (reference "R7") (unit 1) (value "2M") (footprint "Resistor_SMD:R_0603_1608Metric")
     )
     (path "/7132d895-1d0e-496f-8f2c-58a33f44ca13"
-      (reference "R8") (unit 1) (value "2M") (footprint "Resistor_SMD:R_0402_1005Metric")
+      (reference "R8") (unit 1) (value "2M") (footprint "Resistor_SMD:R_0603_1608Metric")
     )
     (path "/b6b8c858-1736-47a7-a5a9-2161c3c217d6"
-      (reference "R9") (unit 1) (value "5.1k") (footprint "Resistor_SMD:R_0402_1005Metric")
+      (reference "R9") (unit 1) (value "5.1k") (footprint "Resistor_SMD:R_0603_1608Metric")
     )
     (path "/63f345a0-ca21-45a2-8405-fdefe13e2ca5"
-      (reference "R10") (unit 1) (value "5.1k") (footprint "Resistor_SMD:R_0402_1005Metric")
+      (reference "R10") (unit 1) (value "5.1k") (footprint "Resistor_SMD:R_0603_1608Metric")
     )
     (path "/90931153-90e4-40c6-a852-f25dc9137e48"

Commit message: Update v1.4
Parts:
- removed J1: ProMicro Pinout, MDBTMicro_library:ProMicro board pinout, symbol MDBTMicro_library:ProMicro
- removed TP10: SWCLK, TestPoint:TestPoint_Pad_D1.0mm, symbol Connector:TestPoint
- removed TP8: GND, TestPoint:TestPoint_Pad_D1.0mm, symbol Connector:TestPoint
- removed TP9: SWDIO, TestPoint:TestPoint_Pad_D1.0mm, symbol Connector:TestPoint
- added J1, J4: Conn_01x13, Connector_PinHeader_2.54mm:PinHeader_1x13_P2.54mm_Vertical, symbol Connector_Generic:Conn_01x13
- added J3: Conn_01x02, Connector_PinHeader_2.54mm:PinHeader_1x02_P2.54mm_Vertical, symbol Connector_Generic:Conn_01x02
Connections:
- net EXT_VCC: now also J4.5 (Pin_5)
- net GND: now also J1.1 (Pin_1), J1.4 (Pin_4), J1.5 (Pin_5), J4.3 (Pin_3)
- net P0.02: now also J4.9 (Pin_9)
- net P0.03: now also J4.11 (Pin_11)
- net P0.06: now also J1.2 (Pin_2)
- net P0.08: now also J1.3 (Pin_3)
- net P0.09: now also J1.11 (Pin_11)
- net P0.10: now also J1.12 (Pin_12)
- net P0.13: now also J1.9 (Pin_9)
- net P0.15: now also J1.6 (Pin_6)
- net P0.17: now also J1.7 (Pin_7)
- net P0.20: now also J1.8 (Pin_8)
- net P0.24: now also J1.10 (Pin_10)
- net P0.28: now also J4.12 (Pin_12)
- net P0.29: now also J4.8 (Pin_8)
- net P0.30: now also J4.6 (Pin_6)
- net P0.31: now also J4.7 (Pin_7)
- net P1.06: now also J1.13 (Pin_13)
- net P1.11: now also J4.13 (Pin_13)
- net P1.13: now also J4.10 (Pin_10)
- net RESET: now also J4.4 (Pin_4)
- net SWCLK: now also J3.2 (Pin_2)
- net SWDIO: now also J3.1 (Pin_1)
- net VBAT: now also J4.1 (Pin_1)
- net VBUS: now also J4.2 (Pin_2)
Other:
- moved on the sheet: C1, C2, C3, C4, D1, J2, JP1, LD1, Q1, Q2, R1, R10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
